Commit message: added rplidar launch and urdf in description, and summit_robot_control

File: summit_description/urdf/summit_rplidar.urdf.xacro (robot description, xacro)
@@ -2,5 +2,5 @@
 <robot name="summit" xmlns:xacro="http://www.ros.org/wiki/xacro">
   <!-- Import all Gazebo-customization elements, including Gazebo colors -->
-  <xacro:include filename="$(find summit_description)/urdf/summit_hokuyo.gazebo" />
+  <xacro:include filename="$(find summit_description)/urdf/summit_rplidar.gazebo" />
   <!-- Robot mechanical and motor parameters -->
   <xacro:property name="PI" value="3.1415926535897931"/>
@@ -444,32 +444,36 @@
   </link>
   <!-- KINECT SENSOR -->
-  <!-- HOKUYO SENSOR -->
-    <link name="hokuyo_base_link">
-      <visual>
-        <origin xyz="0 0 0" rpy="0 0 0"/>
-        <geometry>
-            <mesh filename="package://robotnik_sensors/meshes/hokuyo_utm_30lx.dae"/>
-        </geometry>
-      </visual>
-      <inertial>
-        <mass value="1e-5" />
-        <origin xyz="0 0 0" rpy="0 0 0"/>
-        <inertia ixx="1e-6" ixy="0" ixz="0" iyy="1e-6" iyz="0" izz="1e-6" />
-      </inertial>
-    </link>
-	<link name="hokuyo_link">
+  <!-- RPLIDAR SENSOR -->
+    <link name="rplidar_link">
+		<collision>
+			<origin xyz="0 0 0" rpy="0 0 0"/>
+			<geometry>
+				<box size="0.1 0.1 0.1"/>
+			</geometry>
+		</collision>
+        <visual>
+            <origin xyz="0 0 0" rpy="0 0 0"/>
+            <geometry>
+                <mesh filename="package://robotnik_sensors/meshes/rplidar.dae"/>
+            </geometry>
+        </visual>
+		<!--vision>
+			<origin xyz="0 0 -0.03125" rpy="1.5707 0 0"/>
+			<geometry>
+				<box size="0.1 0.1 0.1"/>
+				<meshfile name="package://robotnik_sensors/meshes/rplidar.dae"/>
+			</geometry>
+		</vision-->
+		<inertial>
+			<mass value="1e-5"/>
+			<origin xyz="0 0 0" rpy="0 0 0"/>
+			<inertia ixx="1e-6" ixy="0" ixz="0" iyy="1e-6" iyz="0" izz="1e-6"/>
+		</inertial>
 	</link>
-    <joint name="hokuyo_joint" type="fixed">
-      <parent link="hokuyo_base_link"/>
-      <child link="hokuyo_link"/>
-      <origin xyz="0.00 0 0.055" rpy="0 0 0"/>
-    </joint>
-  <joint name="hokuyo_base_joint" type="fixed">
-      <!-- FRONT MOUNT  -->
-      <!-- origin xyz="0.29 0 0.1" -->
-      <!-- TOP MOUNT -->
-      <origin xyz="0.0 0.0 0.285"/>
-      <parent link="base_link"/>
-      <child link="hokuyo_base_link"/>
-  </joint>
+	<joint name="rplidar_joint" type="fixed">
+		<axis xyz="0 1 0"/>
+		<origin xyz="0 0 0.22" rpy="0 0 0 "/>
+		<parent link="base_link"/>
+		<child link="rplidar_link"/>
+	</joint>
 </robot>
